File: PCB_kyle/DBF_PCB_ALT_DESIGN/DBF_PCB_ALT_DESIGN.kicad_pcb (KiCad board)
At the start: 4 copper layers, 150 x 65 mm, 7 parts

Commit message: pots
Parts:
- added REF**: B25K, Potentiometer_THT:Potentiometer_Alpha_RD901F-40-00D_Single_Vertical_CircularHoles, F.Cu at (220.8, 87.1)
- added REF**: B25K, Potentiometer_THT:Potentiometer_Alpha_RD901F-40-00D_Single_Vertical_CircularHoles, F.Cu at (220.7, 73.2)
Connections:
- TEENSY pad 21: buzzer -> POT2
- TEENSY pad 22: (no net) -> POT1
- TEENSY pad 23: (no net) -> buzzer
Routing:
- net POT2: track 0.00 -> 32.0 mm
- net POT1: track 0.00 -> 25.0 mm
- net buzzer: track 11.1 -> 14.5 mm

Commit message: Updated DBF_PCB_ALT_DESIGN
Parts:
- added REF**: PinHeader_1x03_P1.00mm_Horizontal, Connector_PinHeader_1.00mm:PinHeader_1x03_P1.00mm_Horizontal, F.Cu at (172.0, 55.4)
- added REF**: PinHeader_1x03_P1.00mm_Horizontal, Connector_PinHeader_1.00mm:PinHeader_1x03_P1.00mm_Horizontal, F.Cu at (181.5, 55.4)
Routing:
- net (no net): vias 0 -> 3
- added copper zone on F.Cu, net GND
Other:
- outline, holes or cut-outs redrawn

Commit message: should be the final thingy
Parts:
- removed the REF** at (220.8, 87.1)
- removed the REF** at (220.7, 73.2)
- moved REF** 57.8 mm to (225.4, 77.5), turned to 180 degrees
- moved REF** 46.9 mm to (225.3, 72.0), turned to 180 degrees
Connections:
- REF** pad 1: (no net) -> GND (x2)
- REF** pad 2: (no net) -> POT2
- REF** pad 3: (no net) -> 5V_PWR (x2)
- REF** pad 2: (no net) -> POT1
Routing:
- net POT2: track 32.0 -> 22.7 mm
- net POT1: track 25.0 -> 24.2 mm
- net GND: vias 4 -> 8
- net 5V_PWR: vias 0 -> 1
- net (no net): vias 3 -> 0
- added copper zone on B.Cu, net 5V_PWR
